Commit message: smaller robot

File: ron_description/urdf/ron_bkp.xacro (robot description, xacro)
@@ -20,7 +20,7 @@
   <xacro:property name="casterMass" value="1"/>
   <xacro:property name="chassisHeight" value="0.5"/>
-  <xacro:property name="chassisLength" value="0.8"/>
-  <xacro:property name="chassisWidth" value="0.5"/>
-  <xacro:property name="chassisMass" value="0.25"/>
+  <xacro:property name="chassisLength" value="1"/>
+  <xacro:property name="chassisWidth" value="1"/>
+  <xacro:property name="chassisMass" value="1"/>
   <xacro:property name="kinect_cam_py" value="-0.0125"/>
   <xacro:property name="cam_px" value="-0.087" />
@@ -73,5 +73,5 @@
   <link name="caster_wheel">
     <collision>
-      <origin xyz="${casterRadius-chassisWidth/2} 0 ${casterRadius}" rpy="0 0 0"/>
+      <origin xyz="${casterRadius-chassisLength/2} 0 ${casterRadius}" rpy="0 0 0"/>
       <geometry>
   <sphere radius="${casterRadius}"/>
@@ -79,5 +79,5 @@
     </collision>
     <visual>
-      <origin xyz="${casterRadius-chassisWidth/2} 0 ${casterRadius}" rpy="0 0 0"/>
+      <origin xyz="${casterRadius-chassisLength/2} 0 ${casterRadius}" rpy="0 0 0"/>
       <geometry>
   <sphere radius="${casterRadius}"/>
@@ -85,10 +85,10 @@
     </visual>
     <inertial>
-      <origin xyz="${casterRadius-chassisWidth/2} 0 ${casterRadius}" rpy="0 0 0"/>
+      <origin xyz="${casterRadius-chassisLength/2} 0 ${casterRadius}" rpy="0 0 0"/>
       <mass value="${casterMass}"/>
       <sphere_inertia m="${casterMass}" r="${casterRadius}"/>
     </inertial>
   </link>
-  <joint name="caster_link" type="fixed">
+  <joint name="fixed" type="fixed">
     <parent link="link1"/>
     <child link="caster_wheel"/>
