Commit message: navigation node

File: ron_description/urdf/ron.xacro (robot description, xacro)
@@ -36,5 +36,5 @@
   <xacro:include filename="$(find ron_description)/urdf/macros.xacro" />
   <!--xacro:include filename="$(find ron_description)/urdf/sensors/kinect.urdf.xacro"/-->
- <link name="base_link" />
+ <link name="base_link"/>
   <joint name="base_joint" type="fixed">
       <parent link="base_link"/>
